File: smolPad.sch (KiCad schematic (older format))
At the start: 25 parts, among them U1 ProMicro

Commit message: Updated design to use both THT and SMD Diodes. Silkscreen added as well.
Parts:
- D1, D10, D11, D12, D2, D3, D4, D5, D6, D7, D8, D9: footprint Diode_SMD:D_SOD-123 -> Keebio-Parts:Diode-dual
Changed lines of the file:
@@
 F 0 "D1" V 5646 3332 50  0000 R CNN
 F 1 "D_Small" V 5555 3332 50  0000 R CNN
-F 2 "Diode_SMD:D_SOD-123" V 5600 3400 50  0001 C CNN
+F 2 "Keebio-Parts:Diode-dual" V 5600 3400 50  0001 C CNN
 F 3 "~" V 5600 3400 50  0001 C CNN
 	1    5600 3400
@@
 F 0 "D2" V 6096 3332 50  0000 R CNN
 F 1 "D_Small" V 6005 3332 50  0000 R CNN
-F 2 "Diode_SMD:D_SOD-123" V 6050 3400 50  0001 C CNN
+F 2 "Keebio-Parts:Diode-dual" V 6050 3400 50  0001 C CNN
 F 3 "~" V 6050 3400 50  0001 C CNN
 	1    6050 3400
@@
 F 0 "D3" V 6546 3332 50  0000 R CNN
 F 1 "D_Small" V 6455 3332 50  0000 R CNN
-F 2 "Diode_SMD:D_SOD-123" V 6500 3400 50  0001 C CNN
+F 2 "Keebio-Parts:Diode-dual" V 6500 3400 50  0001 C CNN
 F 3 "~" V 6500 3400 50  0001 C CNN
 	1    6500 3400
@@
 F 0 "D4" V 5646 3982 50  0000 R CNN
 F 1 "D_Small" V 5555 3982 50  0000 R CNN
-F 2 "Diode_SMD:D_SOD-123" V 5600 4050 50  0001 C CNN
+F 2 "Keebio-Parts:Diode-dual" V 5600 4050 50  0001 C CNN
 F 3 "~" V 5600 4050 50  0001 C CNN
 	1    5600 4050
@@
 F 0 "D5" V 6096 3982 50  0000 R CNN
 F 1 "D_Small" V 6005 3982 50  0000 R CNN
-F 2 "Diode_SMD:D_SOD-123" V 6050 4050 50  0001 C CNN
+F 2 "Keebio-Parts:Diode-dual" V 6050 4050 50  0001 C CNN
 F 3 "~" V 6050 4050 50  0001 C CNN
 	1    6050 4050
@@
 F 0 "D6" V 6546 3982 50  0000 R CNN
 F 1 "D_Small" V 6455 3982 50  0000 R CNN
-F 2 "Diode_SMD:D_SOD-123" V 6500 4050 50  0001 C CNN
+F 2 "Keebio-Parts:Diode-dual" V 6500 4050 50  0001 C CNN
 F 3 "~" V 6500 4050 50  0001 C CNN
 	1    6500 4050
@@
 F 0 "D7" V 5646 4632 50  0000 R CNN
 F 1 "D_Small" V 5555 4632 50  0000 R CNN
-F 2 "Diode_SMD:D_SOD-123" V 5600 4700 50  0001 C CNN
+F 2 "Keebio-Parts:Diode-dual" V 5600 4700 50  0001 C CNN
 F 3 "~" V 5600 4700 50  0001 C CNN
 	1    5600 4700
@@
 F 0 "D8" V 6096 4632 50  0000 R CNN
 F 1 "D_Small" V 6005 4632 50  0000 R CNN
-F 2 "Diode_SMD:D_SOD-123" V 6050 4700 50  0001 C CNN
+F 2 "Keebio-Parts:Diode-dual" V 6050 4700 50  0001 C CNN
 F 3 "~" V 6050 4700 50  0001 C CNN
 	1    6050 4700
@@
 F 0 "D9" V 6546 4632 50  0000 R CNN
 F 1 "D_Small" V 6455 4632 50  0000 R CNN
-F 2 "Diode_SMD:D_SOD-123" V 6500 4700 50  0001 C CNN
+F 2 "Keebio-Parts:Diode-dual" V 6500 4700 50  0001 C CNN
 F 3 "~" V 6500 4700 50  0001 C CNN
 	1    6500 4700
@@
 F 0 "D12" V 6546 5282 50  0000 R CNN
 F 1 "D_Small" V 6455 5282 50  0000 R CNN
-F 2 "Diode_SMD:D_SOD-123" V 6500 5350 50  0001 C CNN
+F 2 "Keebio-Parts:Diode-dual" V 6500 5350 50  0001 C CNN
 F 3 "~" V 6500 5350 50  0001 C CNN
 	1    6500 5350
@@
 F 0 "D11" V 6096 5282 50  0000 R CNN
 F 1 "D_Small" V 6005 5282 50  0000 R CNN
-F 2 "Diode_SMD:D_SOD-123" V 6050 5350 50  0001 C CNN
+F 2 "Keebio-Parts:Diode-dual" V 6050 5350 50  0001 C CNN
 F 3 "~" V 6050 5350 50  0001 C CNN
 	1    6050 5350
@@
 F 0 "D10" V 5646 5282 50  0000 R CNN
 F 1 "D_Small" V 5555 5282 50  0000 R CNN
-F 2 "Diode_SMD:D_SOD-123" V 5600 5350 50  0001 C CNN
+F 2 "Keebio-Parts:Diode-dual" V 5600 5350 50  0001 C CNN
 F 3 "~" V 5600 5350 50  0001 C CNN
 	1    5600 5350
